Commit message: add carto launch and seek link in urdf

File: urdf/dragoon.urdf.xacro (robot description, xacro)
@@ -8,5 +8,4 @@
   </xacro:sensor_d435i>
   <link name="imu_link" />
-  <link name="horizontal_laser_link" />
   <joint name="base_to_imu" type="fixed">
 	  <parent link="base_link"/>
@@ -14,4 +13,5 @@
 	  <origin rpy="0 0 0" xyz="0 0 0"/>
   </joint>
+  <link name="horizontal_laser_link" />
   <joint name="base_to_horizontal_laser_scan" type="fixed">
 	  <parent link="base_link"/>
@@ -19,3 +19,9 @@
 	  <origin rpy="0 0 0" xyz="0 0 0.4"/>
   </joint>
+  <link name="seek_link" />
+  <joint name="base_to_seek" type="fixed">
+	  <parent link="base_link"/>
+	  <child link="seek_link"/>
+	  <origin rpy="0 0 0" xyz="0.2 0.2 0.4"/>
+  </joint>
 </robot>

Commit message: edit urdf after hardware assembly

File: urdf/dragoon.urdf.xacro (robot description, xacro)
@@ -5,5 +5,5 @@
   <link name="base_link" />
   <xacro:sensor_d435i parent="base_link" use_nominal_extrinsics="$(arg use_nominal_extrinsics)">
-    <origin xyz="0.5 0 0.5" rpy="0 0 0"/>
+    <origin xyz="0.001 -0.012 -0.0185" rpy="0 0 0"/>
   </xacro:sensor_d435i>
   <link name="imu_link" />
@@ -11,5 +11,5 @@
 	  <parent link="base_link"/>
 	  <child link="imu_link"/>
-	  <origin rpy="0 0 0" xyz="0 0 0"/>
+	  <origin xyz="0 0 0" rpy="0 0 0" />
   </joint>
   <link name="horizontal_laser_link" />
@@ -17,5 +17,5 @@
 	  <parent link="base_link"/>
 	  <child link="horizontal_laser_link"/>
-	  <origin rpy="0 0 0" xyz="0 0 0.4"/>
+	  <origin xyz="-0.113 0.012 0.13" rpy="0 0 0" />
   </joint>
   <link name="seek_link" />
@@ -23,5 +23,5 @@
 	  <parent link="base_link"/>
 	  <child link="seek_link"/>
-	  <origin rpy="0 0 0" xyz="0.2 0.2 0.4"/>
+	  <origin xyz="-0.0116 0.012 0.078" rpy="0 0 0" />
   </joint>
 </robot>

Commit message: split out bringups, add nav_link

File: urdf/dragoon.urdf.xacro (robot description, xacro)
@@ -7,4 +7,10 @@
     <origin xyz="0.001 -0.012 -0.0185" rpy="0 0 0"/>
   </xacro:sensor_d435i>
+  <link name="nav_link" />
+  <joint name="base_to_nav" type="fixed">
+	  <parent link="base_link"/>
+	  <child link="nav_link"/>
+	  <origin xyz="-0.12 0.012 -0.05" rpy="0 0 0" />
+  </joint>
   <link name="imu_link" />
   <joint name="base_to_imu" type="fixed">
